File: AN-USB-Relay/eagle/01.sch (EAGLE design)
At the start: 18 parts, among them CN2 PIN4, U1 K-09421_AE-BME280, X1 C-07675_USB-B

Commit message: draft
Parts:
- removed U1: K-09421_AE-BME280, 01:K-09421_AE-BME280
- added D1, D2: DIODE, 01:DIODE
- added RL1, RL2: P-09148_ALQ105, 01:P-09148_ALQ105
- added TR1, TR2: I-12467_DTC114EL-T92-K, 01:I-12467_DTC114EL-T92-K
- added U$2, U$3: P-01306_TB111-2-2-U-1-1, Akizuki:P-01306_TB111-2-2-U-1-1
Connections:
- removed net +3V3: C2.2, IC1.VBUS, R6.1, R7.1, U1.VDD
- new net N$13: RL2.NO, U$2.1
- new net N$14: RL1.COM, U$3.2
- new net N$15: RL1.NO, U$3.1
- new net N$17: D2.A, RL2.C2, TR2.C
- new net N$4: C2.2, IC1.VBUS
- new net N$6: D1.A, RL1.C2, TR1.C
- new net N$8: RL2.COM, U$2.2
- net +5V: now also D1.C, D2.C, R6.1, R7.1, RL1.C1, RL2.C1
- net GND: now also TR1.E, TR2.E; no longer U1.GND, U1.SDO
- net GP0: now also TR2.B
- net GP1: now also TR1.B
- net SCL: no longer U1.SCK
- net SDA: no longer U1.SDI
Other:
- note added: "1.0"
- note added: "AN-USB-Relay"
- note added: "ArtifactNoise,LLP / Yuta Kitagami."
- note added: "USB science kit"
- moved on the sheet: CN2, LED1, LED2, LED3, LED4, R10, R11, R6, R7, R8, R9
